Commit message: add marker on top of robot

File: turtlebot3_description/urdf/turtlebot3_burger.urdf.xacro (robot description, xacro)
@@ -31,4 +31,31 @@
     </inertial>
   </link>
+  <link name="aruco_marker_2">
+    <visual>
+      <origin xyz="0 0 0" rpy="0 0 0"/>
+      <geometry>
+        <mesh filename="package://boat_world/models/aruco_marker_2/aruco_marker_2.dae" scale="0.04 0.04 0.04"/>
+      </geometry>
+      <material name="dark"/>
+    </visual>
+    <collision>
+      <origin xyz="0 0 0" rpy="0 0 0"/>
+      <geometry>
+        <mesh filename="package://boat_world/models/aruco_marker_2/aruco_marker_2.dae" scale="0.04 0.04 0.04"/>
+      </geometry>
+    </collision>
+    <inertial>
+      <origin xyz="0 0 0" />
+      <mass value="2.8498940e-02" />
+      <inertia ixx="1.1175580e-05" ixy="-4.2369783e-11" ixz="-5.9381719e-09"
+               iyy="1.1192413e-05" iyz="-1.4400107e-11"
+               izz="2.0712558e-05" />
+      </inertial>
+  </link>
+  <joint name="base_link_to_aruco" type="fixed">
+    <parent link="base_link"/>
+    <child link="aruco_marker_2"/>
+    <origin xyz="-0.03 0 0.19" rpy="0 -1.57 0"/>
+  </joint>
   <joint name="wheel_left_joint" type="continuous">
     <parent link="base_link"/>
